Commit message: update base slam setup
Signed-off-by: Jaeyoung Lee <jylee0121@gmail.com>

File: urdf/udacity_bot.xacro (robot description, xacro)
@@ -191,5 +191,5 @@
       <origin xyz="0 0 0" rpy=" 0 0 0" />
       <geometry>
-        <mesh filename="package://udacity_bot/meshes/hokuyo.dae"/>
+        <mesh filename="package://slam_project/meshes/hokuyo.dae"/>
       </geometry>
     </visual>

Commit message: update robot model
Signed-off-by: Jaeyoung Lee <jylee0121@gmail.com>

File: urdf/udacity_bot.xacro (robot description, xacro)
@@ -1,4 +1,5 @@
 <?xml version='1.0'?>
 <robot name="udacity_bot" xmlns:xacro="http://www.ros.org/wiki/xacro">
+  <xacro:property name="M_PI" value="3.1415926535897931" />
   <xacro:include filename="$(find slam_project)/urdf/udacity_bot.gazebo" />
   <material name="red">
@@ -138,7 +139,7 @@
     <origin xyz="0.2 0 0" rpy="0 0 0" />
     <parent link="chassis" />
-    <child link="camera" />
-  </joint>
-  <link name='camera'>
+    <child link="camera_link" />
+  </joint>
+  <link name='camera_link'>
     <pose>0 0 0 0 0 0</pose>
     <inertial>
@@ -165,4 +166,10 @@
     </visual>
   </link>
+  <joint name="camera_depth_optical_joint" type="fixed">
+    <origin xyz="0 0 0" rpy="${-M_PI/2} 0 ${-M_PI/2}" />
+    <parent link="camera_link" />
+    <child link="camera_rgbd_optical_frame" />
+  </joint>
+  <link name="camera_rgbd_optical_frame"/>
   <!-- LASER RANGEFINDER -->
   <joint name="hokuyo_joint" type="fixed">
